File: schematic/nowcast/nowcast.kicad_sch (KiCad schematic)
At the start: 15 parts, among them J1 Conn_01x05_Pin

Commit message: add silkscreen and edgecuts
Parts:
- removed D14: LED, LED_THT:LED_D5.0mm, symbol Device:LED
- renumbered D2 to D1, D1 to D2
Changed lines of the file:
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@@
   (junction (at 219.71 96.52) (diameter 0) (color 0 0 0 0)
   )
-  (junction (at 251.46 109.22) (diameter 0) (color 0 0 0 0)
-  )
   (junction (at 240.03 121.92) (diameter 0) (color 0 0 0 0)
   )
-  (junction (at 251.46 134.62) (diameter 0) (color 0 0 0 0)
-  )
   (junction (at 210.82 147.32) (diameter 0) (color 0 0 0 0)
   )
@@
     (stroke (width 0) (type default))
   )
-  (wire (pts (xy 251.46 134.62) (xy 260.35 134.62))
-    (stroke (width 0) (type default))
-  )
   (wire (pts (xy 219.71 109.22) (xy 251.46 109.22))
     (stroke (width 0) (type default))
@@
     (stroke (width 0) (type default))
   )
-  (wire (pts (xy 260.35 134.62) (xy 260.35 119.38))
-    (stroke (width 0) (type default))
-  )
   (wire (pts (xy 219.71 134.62) (xy 219.71 137.16))
     (stroke (width 0) (type default))
@@
     (stroke (width 0) (type default))
   )
-  (wire (pts (xy 260.35 109.22) (xy 260.35 111.76))
-    (stroke (width 0) (type default))
-  )
   (wire (pts (xy 231.14 147.32) (xy 240.03 147.32))
     (stroke (width 0) (type default))
@@
   )
   (wire (pts (xy 210.82 121.92) (xy 219.71 121.92))
-    (stroke (width 0) (type default))
-  )
-  (wire (pts (xy 251.46 109.22) (xy 260.35 109.22))
     (stroke (width 0) (type default))
   )
@@
   (symbol (lib_id "Device:LED") (at 219.71 102.87 90) (unit 1)
     (in_bom yes) (on_board yes) (dnp no)
-    (property "Reference" "D1" (at 223.52 100.33 90)
+    (property "Reference" "D2" (at 223.52 100.33 90)
       (effects (font (size 1.27 1.27)) (justify right))
     )
@@
       (project "nowcast"
         (path "/f317fb31-8fcc-4670-94a9-058080a0aa67"
+          (reference "D2") (unit 1)
+        )
+      )
+    )
+  )
+  (symbol (lib_id "Device:LED") (at 231.14 128.27 270) (unit 1)
+    (in_bom yes) (on_board yes) (dnp no)
+    (property "Reference" "D11" (at 234.6325 125.73 90)
+      (effects (font (size 1.27 1.27)))
+    )
+    (property "Value" "LED" (at 234.6325 128.27 90)
+      (effects (font (size 1.27 1.27)))
+    )
+    (property "Footprint" "LED_THT:LED_D5.0mm" (at 231.14 128.27 0)
+      (effects (font (size 1.27 1.27)) hide)
+    )
+    (property "Datasheet" "~" (at 231.14 128.27 0)
+      (effects (font (size 1.27 1.27)) hide)
+    )
+    (pin "1")
+    (pin "2")
+    (instances
+      (project "nowcast"
+        (path "/f317fb31-8fcc-4670-94a9-058080a0aa67"
+          (reference "D11") (unit 1)
+        )
+      )
+    )
+  )
+  (symbol (lib_id "Device:LED") (at 251.46 115.57 270) (unit 1)
+    (in_bom yes) (on_board yes) (dnp no)
+    (property "Reference" "D13" (at 254.9525 113.03 90)
+      (effects (font (size 1.27 1.27)))
+    )
+    (property "Value" "LED" (at 254.9525 115.57 90)
+      (effects (font (size 1.27 1.27)))
+    )
+    (property "Footprint" "LED_THT:LED_D5.0mm" (at 251.46 115.57 0)
+      (effects (font (size 1.27 1.27)) hide)
+    )
+    (property "Datasheet" "~" (at 251.46 115.57 0)
+      (effects (font (size 1.27 1.27)) hide)
+    )
+    (pin "1")
+    (pin "2")
+    (instances
+      (project "nowcast"
+        (path "/f317fb31-8fcc-4670-94a9-058080a0aa67"
+          (reference "D13") (unit 1)
+        )
+      )
+    )
+  )
+  (symbol (lib_id "Device:LED") (at 210.82 102.87 270) (unit 1)
+    (in_bom yes) (on_board yes) (dnp no)
+    (property "Reference" "D1" (at 214.3125 100.33 90)
+      (effects (font (size 1.27 1.27)))
+    )
+    (property "Value" "LED" (at 214.3125 102.87 90)
+      (effects (font (size 1.27 1.27)))
+    )
+    (property "Footprint" "LED_THT:LED_D5.0mm" (at 210.82 102.87 0)
+      (effects (font (size 1.27 1.27)) hide)
+    )
+    (property "Datasheet" "~" (at 210.82 102.87 0)
+      (effects (font (size 1.27 1.27)) hide)
+    )
+    (pin "1")
+    (pin "2")
+    (instances
+      (project "nowcast"
+        (path "/f317fb31-8fcc-4670-94a9-058080a0aa67"
           (reference "D1") (unit 1)
         )
@@
     )
   )
-  (symbol (lib_id "Device:LED") (at 231.14 128.27 270) (unit 1)
-    (in_bom yes) (on_board yes) (dnp no)
-    (property "Reference" "D11" (at 234.6325 125.73 90)
-      (effects (font (size 1.27 1.27)))
-    )
-    (property "Value" "LED" (at 234.6325 128.27 90)
-      (effects (font (size 1.27 1.27)))
-    )
-    (property "Footprint" "LED_THT:LED_D5.0mm" (at 231.14 128.27 0)
-      (effects (font (size 1.27 1.27)) hide)
-    )
-    (property "Datasheet" "~" (at 231.14 128.27 0)
-      (effects (font (size 1.27 1.27)) hide)
-    )
-    (pin "1")
-    (pin "2")
-    (instances
-      (project "nowcast"
-        (path "/f317fb31-8fcc-4670-94a9-058080a0aa67"
-          (reference "D11") (unit 1)
-        )
-      )
-    )
-  )
-  (symbol (lib_id "Device:LED") (at 251.46 115.57 270) (unit 1)
-    (in_bom yes) (on_board yes) (dnp no)
-    (property "Reference" "D13" (at 254.9525 113.03 90)
-      (effects (font (size 1.27 1.27)))
-    )
-    (property "Value" "LED" (at 254.9525 115.57 90)
-      (effects (font (size 1.27 1.27)))
-    )
-    (property "Footprint" "LED_THT:LED_D5.0mm" (at 251.46 115.57 0)
-      (effects (font (size 1.27 1.27)) hide)
-    )
-    (property "Datasheet" "~" (at 251.46 115.57 0)
-      (effects (font (size 1.27 1.27)) hide)
-    )
-    (pin "1")
-    (pin "2")
-    (instances
-      (project "nowcast"
-        (path "/f317fb31-8fcc-4670-94a9-058080a0aa67"
-          (reference "D13") (unit 1)
-        )
-      )
-    )
-  )
-  (symbol (lib_id "Device:LED") (at 210.82 102.87 270) (unit 1)
-    (in_bom yes) (on_board yes) (dnp no)
-    (property "Reference" "D2" (at 214.3125 100.33 90)
-      (effects (font (size 1.27 1.27)))
-    )
-    (property "Value" "LED" (at 214.3125 102.87 90)
-      (effects (font (size 1.27 1.27)))
-    )
-    (property "Footprint" "LED_THT:LED_D5.0mm" (at 210.82 102.87 0)
-      (effects (font (size 1.27 1.27)) hide)
-    )
-    (property "Datasheet" "~" (at 210.82 102.87 0)
-      (effects (font (size 1.27 1.27)) hide)
-    )
-    (pin "1")
-    (pin "2")
-    (instances
-      (project "nowcast"
-        (path "/f317fb31-8fcc-4670-94a9-058080a0aa67"
-          (reference "D2") (unit 1)
-        )
-      )
-    )
-  )
   (symbol (lib_id "Device:LED") (at 240.03 128.27 90) (unit 1)
     (in_bom yes) (on_board yes) (dnp no)
@@
         )
       )
-    )
-  )
-  (symbol (lib_id "Device:LED") (at 260.35 115.57 90) (unit 1)
-    (in_bom yes) (on_board yes) (dnp no)
-    (property "Reference" "D14" (at 264.16 113.03 90)
-      (effects (font (size 1.27 1.27)) (justify right))
-    )
-    (property "Value" "LED" (at 264.16 115.57 90)
-      (effects (font (size 1.27 1.27)) (justify right))
-    )
-    (property "Footprint" "LED_THT:LED_D5.0mm" (at 260.35 115.57 0)
-      (effects (font (size 1.27 1.27)) hide)
-    )
-    (property "Datasheet" "~" (at 260.35 115.57 0)
-      (effects (font (size 1.27 1.27)) hide)
-    )
-    (pin "1")
-    (pin "2")
-    (instances
-      (project "nowcast"
-        (path "/f317fb31-8fcc-4670-94a9-058080a0aa67"
-          (reference "D14") (unit 1)
-        )
-      )
