File: schematic/nowcast/nowcast.kicad_pcb (KiCad board)
At the start: 2 copper layers, 15 parts, among them J1 Conn_01x05_Pin

Commit message: add silkscreen and edgecuts
Parts:
- removed D14: LED, LED_THT:LED_D5.0mm
- moved D1 879.9 mm to (550.6, 783.8)
- moved D2 828.8 mm to (496.1, 763.5)
- moved J1 801.3 mm to (585.7, 786.1), turned to -90 degrees
- moved D3 777.6 mm to (448.6, 730.5)
- moved D4 713.4 mm to (409.9, 687.3)
- moved D5 646.4 mm to (382.8, 636.3)
- moved D6 577.5 mm to (369.7, 579.5)
- moved D7 512.4 mm to (369.3, 521.8)
- moved D8 454.7 mm to (383.2, 465.9)
- moved D13 434.2 mm to (611.1, 339.1)
- moved D9 409.1 mm to (410.0, 415.2)
- moved D10 379.8 mm to (448.8, 371.0)
- moved D12 353.6 mm to (549.8, 317.7)
- moved D11 303.9 mm to (496.3, 338.5)
- renumbered D2 to D1, D1 to D2
Other:
- board outline added: 240 x 518.5 mm

Commit message: adjusted pcb design
Parts:
- moved D4 321.5 mm to (730.1, 715.1)
- moved D5 320.6 mm to (701.6, 669.6)
- moved D3 320.3 mm to (768.1, 753.0)
- moved D2 318.2 mm to (813.7, 781.8)
- moved D6 316.6 mm to (683.9, 618.8)
- moved D1 314.1 mm to (864.4, 799.4)
- moved D7 311.6 mm to (677.8, 565.4)
- moved J1 311.2 mm to (896.2, 806.8)
- moved D8 304.1 mm to (683.8, 511.9)
- moved D9 295.2 mm to (701.6, 461.2)
- moved D10 284.9 mm to (730.1, 415.7)
- moved D11 274.6 mm to (768.1, 377.8)
- moved D12 265.8 mm to (813.7, 349.1)
- moved D13 253.4 mm to (864.4, 331.4)
Routing:
- net NOWCAST_D: track 0.00 -> 705.3 mm
- net NOWCAST_B: track 0.00 -> 694.7 mm
- net NOWCAST_C: track 0.00 -> 655.4 mm
- net NOWCAST_E: track 0.00 -> 652.8 mm
- net NOWCAST_A: track 0.00 -> 553.8 mm
- added copper zone on B.Cu, net (none)
- added copper zone on F.Cu, net (none)
